File: bike_light_pcb/bike_light_pcb.sch (KiCad schematic (older format))
At the start: 9 parts, among them J1 Conn_01x03_Male, J2 Conn_01x04_Female, J3 Conn_01x02_Female, U1 Teensy4.0, U2 HM18_BLE, U3 MPU605, U4 charge_module

Commit message: draft 1 schem
Parts:
- added BT?: Battery_Cell, symbol Device:Battery_Cell
- added J?: USB_B_Micro_Charge, symbol Connector:USB_B_Micro
Connections:
- net 5V_VUSB is gone; now on net 5V_MAIN: SW?.2 (B)
- net 5V_CHRG: now also J?.1 (Pin_1), J?.1 (VBUS); no longer SW?.1 (A)
- net 5V_MAIN: now also J1.1 (Pin_1), J3.1 (Pin_1), U3.1 (VCC); no longer SW?.3 (C), U1.33 (VIN)
- net 5V_MODULE: now also SW?.1 (A); no longer SW?.4 (A)
- net GND_CHRG: now also J?.2 (Pin_2), J?.5 (GND)
- net GND_MAIN: now also J1.3 (Pin_3), J3.2 (Pin_2), SW?.5 (B), U1.17 (GND), U1.32 (GND), U1.47 (GND), U3.2 (GND)
- net GND_MODULE: now also SW?.4 (A)
- net at U2.3 (TXD): now also U1.3 (1_TX1_CTX2_MISO1)
- net at U2.4 (RXD): now also U1.2 (0_RX1_CRX2_CS1)
- net at U3.3 (SCL): now also U1.26 (19_A5_SCL0)
- net at U3.4 (SDA): now also U1.25 (18_A4_SDA0)
- net at U3.8 (INT): now also U1.22 (15_A1_RX3_SPDIF_IN)
- net at U1.10 (8_TX2_IN1): now also J2.1 (Pin_1)
- net CHRG_KEY: now reaches U1.11 (9_OUT1C)
- net CHRG_KEY: now also U4.7 (KEY)
- net RGB_D: now reaches U1.27 (20_A6_TX5_LRCLK1)
- net RGB_D: now also J1.2 (Pin_2)
- net at U1.6 (4_BCLK2): now also J2.4 (Pin_4)
- net at U1.7 (5_IN2): now also J2.3 (Pin_3)
- net at U1.9 (7_RX2_OUT1A): now also J2.2 (Pin_2)
- net at U4.3 (GND_BATT): now also BT?.2 (-)
- net at U4.4 (VIN_BATT): now also BT?.1 (+)
- net 5V_USB renamed TEENSY_VUSB
- net TEENSY_VUSB: now also SW?.3 (C); no longer SW?.5 (B)
- no-connect marks 0 -> 47
Other:
- note added: "1. Everything running on battery power\n2. Battery power disconnected. Usb plugged into teensy powerning everything."
- note removed: "Cut VIN-VUSB trace"
- note removed: "Modes\n1. plug in usb to charge\n2. plug in usb to program\n3. run off of battery\n"
- moved on the sheet: J1, J2, J3, J?, SW?, U1, U2, U3, U4
